Commit message: feat:添加4pro机器人的ik-fast文件以及工作空间输出结果

File: src/biped_s42/urdf/biped_s42.urdf (robot description, URDF)
Before this commit: robot biped_s42, 26 links, 25 joints
Links:
- link base_link: geometry collision mesh filename=package://biped_s42/meshes/HEAD_URDF.STL; visual mesh filename=package://biped_s42/meshes/HEAD_URDF.STL

File: src/biped_s42/urdf/biped_s42_with_v4_arm.urdf (robot description, URDF)
Before this commit: robot biped_s42, 42 links, 41 joints
Links:
- link base_link: geometry collision mesh filename=package://biped_s42/meshes/HEAD_URDF.STL; visual mesh filename=package://biped_s42/meshes/HEAD_URDF.STL
